File: JTAG_Breakout.kicad_pcb (KiCad board)
At the start: 2 copper layers, 21 x 23 mm, 2 parts, among them J1 JTAG_IN, J2 Breakout

Commit message: Fab this board, edits by Keith
Parts:
- added G***: LOGO, Coolsilks:allison_silk_pretty, B.Cu at (119.5, 104.7)
- moved J2 15.4 mm to (123.8, 91.4), turned to 0 degrees
- moved J1 12.7 mm to (115.6, 105.1), turned to 180 degrees
Routing:
- net /TDO: track 8.43 -> 38.5 mm
- net GND: track 27.2 -> 0.00 mm
- net /TCK: track 8.26 -> 32.2 mm
- net /TDI: track 8.66 -> 31.7 mm
- net /TMS: track 8.49 -> 25.5 mm
- net /PS_SRST_B: track 9.10 -> 16.0 mm
- net /VCCO_0: track 8.71 -> 15.4 mm
- added copper zone on B.Cu, net GND
Other:
- board text added: "Breakout"
- board text added: "JTAG cable"
- board text added: "PS_SRST_B, X, TDI, TDO, TCK, TMS, VCC_O"
- board text added: "Top - GND"
